File: Hardware/SparkFun_LilyPad-Button.brd (EAGLE design)
At the start: 7.6 x 15.6 mm, 5 parts

Commit message: Initial Commit
Parts:
- removed BUTTON-, BUTTONS: SEWTAP8, LilyPad-Wearables:PETAL-MEDIUM-2SIDE
- removed LOGO1: LOGO-LPL, LilyPad-Wearables:LOGO-L
- removed S1: (no value), SparkFun:TACTILE_SWITCH_SMD
- added FRAME2: FRAME-LETTER, SparkFun-Aesthetics:CREATIVE_COMMONS
- added JP12, JP13: SEWTAP_MEDIUM-2SIDE, LilyPad-Wearables:PETAL-MEDIUM-2SIDE
- added S4: MOMENTARY-SWITCH-SPST-SMD-5.2-REDUNDANT, SparkFun-Switches:TACTILE_SWITCH_SMD_5.2MM
- added U$45: (no value), LilyPad-Wearables:LOGO-L
- U$1: value CREATIVE_COMMONS -> SPECIAL_INSTRUCTIONS-ORDERING; device SparkFun:CREATIVE_COMMONS -> SparkFun-Aesthetics:ORDERING_INSTRUCTIONS
- moved U$1 12.7 mm to (-19.1, -24.1)
Connections:
- removed net -: BUTTON-.1, S1.4
- removed net S: BUTTONS.1, S1.2
- new net D4: JP12.1, S4.1, S4.2
- new net GND: JP13.1, S4.3, S4.4
Routing:
- net D4: track 0.00 -> 16.4 mm, vias 0 -> 1
- net GND: track 0.00 -> 14.4 mm, vias 0 -> 1
- net S: track 4.58 -> 0.00 mm
- net -: track 4.58 -> 0.00 mm
Other:
- board size 7.6 x 15.6 mm -> 15.7 x 8 mm
- board text added: "Button"
- board text added: "Elias Santistevan"
- board text added: "Finishing: Lead-free HASL"
- board text added: "LilyPad concept and shapes by: L. Buechley and N. Seidle"
- board text added: "Marshal Taylor"
- board text added: "Marshall Taylor"
- board text added: "PCB thickness: 31 mil / 0.8mm"
- board text added: "Plated holes: 0.013 0.026 0.0276 0.0866 0.11 0.1575"
- board text added: "Revised by:"
- board text added: "Revised by: Elias Santistevan"
- board text added: "Solder mask color: Purple (Lilypad)"
- board text added: "Unplated holes: 0.015 0.02 0.315 0.0335"
- board text added: "v13"
- board text removed: "-"
- board text removed: "S"
