File: Production/SparkFun_LilyPad-Button-Panel_v20.brd (EAGLE design)
At the start: 138.7 x 252.7 mm, 703 parts

Commit message: updated v20 panel with new silk
Parts:
- moved JP11 24.6 mm to (12.2, 36.4)
- moved JP14 24.6 mm to (19.8, 36.4)
- moved S7 24.6 mm to (16.0, 36.4)
- moved U$6 24.6 mm to (16.0, 36.3), turned to 0 degrees
- moved U$3 24.6 mm to (33.8, 19.4), turned to 0 degrees
- moved JP5 24.5 mm to (30.0, 19.4)
- moved JP6 24.5 mm to (37.6, 19.4)
- moved S3 24.5 mm to (33.8, 19.4)
- moved JP17 19.7 mm to (12.2, 44.8)
- moved JP18 19.7 mm to (19.8, 44.8)
- moved S9 19.7 mm to (16.0, 44.8)
- moved U$8 19.7 mm to (16.0, 44.8), turned to 0 degrees
- moved U$1 19.7 mm to (33.8, 10.9), turned to 0 degrees
- moved JP1 19.7 mm to (30.0, 10.9)
- moved JP2 19.7 mm to (37.6, 10.9)
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Other:
- outline, holes or cut-outs redrawn
